File: docs/oruga_board.kicad_sch (KiCad schematic)
At the start: 13 parts, among them J1 UART CONSOLE, J3 I2CBus, M1 M1, M2 M2, M3 M3, M4 M4

Commit message: chore(docs): update schematics
Parts:
- added SW1: SW_Push, symbol Switch:SW_Push
- renumbered U1 to GPIO04
Connections:
- net GND: now also SW1.1
- net ESTOP: now reaches GPIO04.13 (GPIO04)
- net ESTOP: now also U2. (M2B), SW1.2
- no-connect marks 26 -> 24
Changed lines of the file:
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@@
 (kicad_sch
-	(version 20231120)
+	(version 20250114)
 	(generator "eeschema")
-	(generator_version "8.0")
+	(generator_version "9.0")
 	(paper "A4")
 	(junction
@@
 	)
 	(no_connect
-		(at 72.39 93.98)
-	)
-	(no_connect
 		(at 35.56 86.36)
 	)
@@
 	)
 	(no_connect
-		(at 35.56 81.28)
-	)
-	(no_connect
 		(at 116.84 48.26)
 	)
@@
 	(wire
 		(pts
+			(xy 214.63 115.57) (xy 208.28 115.57)
+		)
+		(stroke
+			(width 0)
+			(type default)
+		)
+	)
+	(wire
+		(pts
 			(xy 237.49 96.52) (xy 242.57 96.52)
 		)
@@
 	(wire
 		(pts
+			(xy 229.87 96.52) (xy 229.87 105.41)
+		)
+		(stroke
+			(width 0)
+			(type default)
+		)
+	)
+	(wire
+		(pts
 			(xy 106.68 50.8) (xy 116.84 50.8)
 		)
@@
 	(wire
 		(pts
+			(xy 26.67 81.28) (xy 35.56 81.28)
+		)
+		(stroke
+			(width 0)
+			(type default)
+		)
+	)
+	(wire
+		(pts
 			(xy 72.39 60.96) (xy 81.28 60.96)
 		)
@@
 		)
 	)
+	(label "ESTOP"
+		(at 229.87 96.52 270)
+		(effects
+			(font
+				(size 1.27 1.27)
+			)
+			(justify right bottom)
+		)
+	)
 	(label "SCL"
 		(at 81.28 60.96 180)
@@
 		)
 	)
+	(label "ESTOP"
+		(at 26.67 81.28 0)
+		(effects
+			(font
+				(size 1.27 1.27)
+			)
+			(justify left bottom)
+		)
+	)
 	(label "M2B"
 		(at 240.03 133.35 90)
@@
 		)
 	)
+	(label "ESTOP"
+		(at 214.63 115.57 180)
+		(effects
+			(font
+				(size 1.27 1.27)
+			)
+			(justify right bottom)
+		)
+	)
 	(label "CONS_TX"
 		(at 106.68 53.34 0)
@@
 		)
 		(instances
-			(project ""
+			(project "oruga_board"
 				(path "/53598eb1-4760-44d6-8482-68cc5e5a205e"
 					(reference "M1")
@@
 		)
 		(instances
-			(project ""
+			(project "oruga_board"
 				(path "/53598eb1-4760-44d6-8482-68cc5e5a205e"
 					(reference "#PWR03")
@@
 		)
 		(instances
-			(project ""
+			(project "oruga_board"
 				(path "/53598eb1-4760-44d6-8482-68cc5e5a205e"
 					(reference "D1")
@@
 		(dnp no)
 		(fields_autoplaced yes)
-		(property "Reference" "U1"
+		(property "Reference" "GPIO04"
 			(at 53.975 40.64 0)
 			(effects
@@
 		)
 		(instances
-			(project ""
+			(project "oruga_board"
 				(path "/53598eb1-4760-44d6-8482-68cc5e5a205e"
-					(reference "U1")
+					(reference "GPIO04")
 					(unit 1)
 				)
@@
 		)
 		(instances
-			(project ""
+			(project "oruga_board"
 				(path "/53598eb1-4760-44d6-8482-68cc5e5a205e"
 					(reference "#PWR07")
@@
 	)
 	(symbol
+		(lib_id "Switch:SW_Push")
+		(at 203.2 115.57 0)
+		(unit 1)
+		(exclude_from_sim no)
+		(in_bom yes)
+		(on_board yes)
+		(dnp no)
+		(fields_autoplaced yes)
+		(property "Reference" "SW1"
+			(at 203.2 107.95 0)
+			(effects
+				(font
+					(size 1.27 1.27)
+				)
+			)
+		)
+		(property "Value" "SW_Push"
+			(at 203.2 110.49 0)
+			(effects
+				(font
+					(size 1.27 1.27)
+				)
+			)
+		)
+		(property "Footprint" ""
+			(at 203.2 110.49 0)
+			(effects
+				(font
+					(size 1.27 1.27)
+				)
+				(hide yes)
+			)
+		)
+		(property "Datasheet" "~"
+			(at 203.2 110.49 0)
+			(effects
+				(font
+					(size 1.27 1.27)
+				)
+				(hide yes)
+			)
+		)
+		(property "Description" "Push button switch, generic, two pins"
+			(at 203.2 115.57 0)
+			(effects
+				(font
+					(size 1.27 1.27)
+				)
+				(hide yes)
+			)
+		)
+		(pin "2"
+		)
+		(pin "1"
+		)
+		(instances
+			(project "oruga_board"
+				(path "/53598eb1-4760-44d6-8482-68cc5e5a205e"
+					(reference "SW1")
+					(unit 1)
+				)
+			)
+		)
+	)
+	(symbol
 		(lib_id "power:GND")
 		(at 104.14 100.33 0)
@@
 		)
 		(instances
-			(project ""
+			(project "oruga_board"
 				(path "/53598eb1-4760-44d6-8482-68cc5e5a205e"
 					(reference "#PWR08")
@@
 		)
 		(instances
-			(project ""
+			(project "oruga_board"
 				(path "/53598eb1-4760-44d6-8482-68cc5e5a205e"
 					(reference "#PWR015")
@@
 		)
 		(instances
-			(project ""
+			(project "oruga_board"
 				(path "/53598eb1-4760-44d6-8482-68cc5e5a205e"
 					(reference "#PWR02")
@@
 		)
 		(instances
-			(project ""
+			(project "oruga_board"
 				(path "/53598eb1-4760-44d6-8482-68cc5e5a205e"
 					(reference "M3")
@@
 	)
 	(symbol
+		(lib_id "power:GND")
+		(at 198.12 115.57 0)
+		(unit 1)
+		(exclude_from_sim no)
+		(in_bom yes)
+		(on_board yes)
+		(dnp no)
+		(fields_autoplaced yes)
+		(property "Reference" "#PWR017"
+			(at 198.12 121.92 0)
+			(effects
+				(font
+					(size 1.27 1.27)
+				)
+				(hide yes)
+			)
+		)
+		(property "Value" "GND"
+			(at 198.12 120.65 0)
+			(effects
+				(font
+					(size 1.27 1.27)
+				)
+			)
+		)
+		(property "Footprint" ""
+			(at 198.12 115.57 0)
+			(effects
+				(font
+					(size 1.27 1.27)
+				)
+				(hide yes)
+			)
+		)
+		(property "Datasheet" ""
+			(at 198.12 115.57 0)
+			(effects
+				(font
+					(size 1.27 1.27)
+				)
+				(hide yes)
+			)
+		)
+		(property "Description" "Power symbol creates a global label with name \"GND\" , ground"
+			(at 198.12 115.57 0)
+			(effects
+				(font
+					(size 1.27 1.27)
+				)
+				(hide yes)
+			)
+		)
+		(pin "1"
+		)
+		(instances
+			(project "oruga_board"
+				(path "/53598eb1-4760-44d6-8482-68cc5e5a205e"
+					(reference "#PWR017")
+					(unit 1)
+				)
+			)
+		)
+	)
+	(symbol
 		(lib_id "power:+3.3V")
 		(at 64.77 129.54 0)
@@
 		)
 		(instances
-			(project ""
+			(project "oruga_board"
 				(path "/53598eb1-4760-44d6-8482-68cc5e5a205e"
 					(reference "J3")
@@
 		)
 		(instances
-			(project ""
+			(project "oruga_board"
 				(path "/53598eb1-4760-44d6-8482-68cc5e5a205e"
 					(reference "U2")
@@
 		)
 		(instances
-			(project ""
+			(project "oruga_board"
 				(path "/53598eb1-4760-44d6-8482-68cc5e5a205e"
 					(reference "J1")
@@
 		)
 		(instances
-			(project ""
+			(project "oruga_board"
 				(path "/53598eb1-4760-44d6-8482-68cc5e5a205e"
 					(reference "#PWR09")
@@
 		)
 		(instances
-			(project ""
+			(project "oruga_board"
 				(path "/53598eb1-4760-44d6-8482-68cc5e5a205e"
 					(reference "R1")
@@
 		)
 		(instances
-			(project ""
+			(project "oruga_board"
 				(path "/53598eb1-4760-44d6-8482-68cc5e5a205e"
 					(reference "BT1")
@@
 		)
 	)
+	(embedded_fonts no)
 )
